File: proto 6x.kicad_pcb (KiCad board)
At the start: 2 copper layers, 84 parts

Commit message: fix bottom row, not yet fixed arrow keys
Parts:
- moved REF**21 4.73 mm to (412.3, 132.9)
- moved REF**21 4.55 mm to (393.2, 113.8)
- moved REF**21 4.39 mm to (393.3, 132.9)
- moved REF**21 4.20 mm to (374.3, 132.9)
- moved REF** 3.76 mm to (231.8, 127.0)
- moved REF** 3.75 mm to (150.8, 127.0)
- moved REF** 3.75 mm to (341.3, 127.0)
- moved REF** 3.75 mm to (312.7, 127.0)
- moved REF** 3.57 mm to (122.2, 127.0)

Commit message: fix arrow keys, add split bs, stepped caps lock, basic board outline
Parts:
- added REF**: 1U, MX_Only:MXOnly-1.25U-Hotswap, F.Cu at (119.9, 88.9)
- added REF**: 2U, MX_Only:MXOnly-2U-Hotswap, F.Cu at (374.6, 50.8)
- moved REF**21 4.57 mm to (369.9, 131.7)
- moved REF**21 4.52 mm to (388.9, 131.7)
- moved REF**21 4.48 mm to (408.0, 131.7)
- moved REF**21 4.46 mm to (388.9, 112.6)
- turned REF** to 180 degrees
- turned REF**13 to 180 degrees
- turned REF**14 to 180 degrees
Other:
- board outline added: 405.1 x 105.1 mm

Commit message: basic board pcb layout
Parts:
- added REF**: 2U, MX_Only:MXOnly-2U-ReversedStabilizers-NoLED, F.Cu at (60.3, 127.0)
- added REF**: 2U, MX_Only:MXOnly-2U-ReversedStabilizers-NoLED, F.Cu at (79.4, 127.0)
- added REF**: D_SOD-323F, Diode_SMD:D_SOD-323F, F.Cu at (47.7, 51.1)
- added REF**: 7U, MX_Only:MXOnly-6.25U-ReversedStabilizers-NoLED, F.Cu at (238.9, 127.0)
- added REF**: D_SOD-323F, Diode_SMD:D_SOD-323F, F.Cu at (119.2, 70.1)
- added REF**: 1U, MX_Only:MXOnly-1.25U-NoLED, F.Cu at (119.9, 127.0)
- added REF**: D_SOD-323F, Diode_SMD:D_SOD-323F, F.Cu at (114.4, 51.1)
- added REF**11: 1U, MX_Only:MXOnly-1U-NoLED, F.Cu at (360.4, 88.9)
- added REF**11: 1U, MX_Only:MXOnly-1U-NoLED, F.Cu at (141.3, 108.0)
- added REF**29: 1U, MX_Only:MXOnly-1.25U-NoLED, F.Cu at (143.7, 127.0)
- added REF**30: 1U, MX_Only:MXOnly-1.25U-NoLED, F.Cu at (167.5, 127.0)
- added REF**30: 1U, MX_Only:MXOnly-1.25U-NoLED, F.Cu at (381.8, 88.9)
- added REF**30: 1U, MX_Only:MXOnly-1.25U-NoLED, F.Cu at (119.9, 108.0)
- added REF**31: 1U, MX_Only:MXOnly-1U-NoLED, F.Cu at (327.0, 127.0)
- added REF**32: 1U, MX_Only:MXOnly-1U-NoLED, F.Cu at (346.1, 127.0)
- added REF**33: D_SOD-323F, Diode_SMD:D_SOD-323F, F.Cu at (133.4, 51.1)
- added REF**34: D_SOD-323F, Diode_SMD:D_SOD-323F, F.Cu at (152.5, 51.1)
- added REF**35: D_SOD-323F, Diode_SMD:D_SOD-323F, F.Cu at (171.5, 51.1)
- added REF**36: D_SOD-323F, Diode_SMD:D_SOD-323F, F.Cu at (190.6, 51.1)
- added REF**37: D_SOD-323F, Diode_SMD:D_SOD-323F, F.Cu at (209.6, 51.1)
- added REF**38: D_SOD-323F, Diode_SMD:D_SOD-323F, F.Cu at (228.7, 51.1)
- added REF**39: D_SOD-323F, Diode_SMD:D_SOD-323F, F.Cu at (247.7, 51.1)
- added REF**40: D_SOD-323F, Diode_SMD:D_SOD-323F, F.Cu at (266.8, 51.1)
- added REF**41: D_SOD-323F, Diode_SMD:D_SOD-323F, F.Cu at (285.8, 51.1)
- added REF**42: D_SOD-323F, Diode_SMD:D_SOD-323F, F.Cu at (304.9, 51.1)
- added REF**43: D_SOD-323F, Diode_SMD:D_SOD-323F, F.Cu at (323.9, 51.1)
- added REF**44: D_SOD-323F, Diode_SMD:D_SOD-323F, F.Cu at (343.0, 51.1)
- added REF**44: D_SOD-323F, Diode_SMD:D_SOD-323F, F.Cu at (409.7, 51.1)
- added REF**45: D_SOD-323F, Diode_SMD:D_SOD-323F, F.Cu at (66.8, 51.1)
- added REF**46: D_SOD-323F, Diode_SMD:D_SOD-323F, F.Cu at (85.8, 51.1)
- added REF**47: D_SOD-323F, Diode_SMD:D_SOD-323F, F.Cu at (47.7, 70.1)
- added REF**48: D_SOD-323F, Diode_SMD:D_SOD-323F, F.Cu at (66.8, 70.1)
- added REF**49: D_SOD-323F, Diode_SMD:D_SOD-323F, F.Cu at (85.8, 70.1)
- added REF**50: D_SOD-323F, Diode_SMD:D_SOD-323F, F.Cu at (47.7, 89.2)
- added REF**51: D_SOD-323F, Diode_SMD:D_SOD-323F, F.Cu at (66.8, 89.2)
- added REF**52: D_SOD-323F, Diode_SMD:D_SOD-323F, F.Cu at (85.8, 89.2)
- added REF**53: D_SOD-323F, Diode_SMD:D_SOD-323F, F.Cu at (47.7, 108.2)
- added REF**54: D_SOD-323F, Diode_SMD:D_SOD-323F, F.Cu at (66.8, 108.2)
- added REF**55: D_SOD-323F, Diode_SMD:D_SOD-323F, F.Cu at (85.8, 108.2)
- added REF**56: D_SOD-323F, Diode_SMD:D_SOD-323F, F.Cu at (409.7, 70.1)
- added REF**57: D_SOD-323F, Diode_SMD:D_SOD-323F, F.Cu at (409.7, 89.2)
- added REF**58: D_SOD-323F, Diode_SMD:D_SOD-323F, F.Cu at (428.7, 51.1)
- added REF**59: D_SOD-323F, Diode_SMD:D_SOD-323F, F.Cu at (428.7, 70.1)
- added REF**60: D_SOD-323F, Diode_SMD:D_SOD-323F, F.Cu at (428.7, 89.2)
- added REF**8: 1U, MX_Only:MXOnly-1U-NoLED, F.Cu at (308.0, 127.0)
- added U1: W25Q128JVS, Package_SO:SOIC-8_5.23x5.23mm_P1.27mm, B.Cu at (433.8, 108.5)
- added U3: RP2040, Sleep-Lib:RP2040-QFN-56, B.Cu at (421.8, 110.3)
- added USB1: HRO-TYPE-C-31-M-12, Type-C:HRO-TYPE-C-31-M-12-Assembly, B.Cu at (398.5, 35.6)
- added Y1: 12MHz, Crystal:Crystal_SMD_3225-4Pin_3.2x2.5mm, B.Cu at (430.1, 120.9)
- REF** (x5), REF**13: footprint MX_Only:MXOnly-1.5U-Hotswap -> MX_Only:MXOnly-1.5U-NoLED
- REF** (x3), REF**1 (x4), REF**10 (x4), REF**11 (x3), REF**12 (x2), REF**13, REF**14, REF**15 (x2), REF**16, REF**17 (x2), REF**18 (x2), REF**19, REF**2 (x4), REF**20 (x2), REF**21 (x6), REF**22, REF**23, REF**24, REF**25, REF**26, REF**27, REF**28, REF**3 (x4), REF**4 (x4), REF**5 (x4), REF**6 (x4), REF**7 (x4), REF**8 (x4), REF**9 (x4): footprint MX_Only:MXOnly-1U-Hotswap -> MX_Only:MXOnly-1U-NoLED
- REF** (x2): footprint MX_Only:MXOnly-1.75U-Hotswap -> MX_Only:MXOnly-1.75U-NoLED
- REF**: footprint MX_Only:MXOnly-2.25U-Hotswap -> MX_Only:MXOnly-2.25U-NoLED
- REF**: footprint MX_Only:MXOnly-1.25U-Hotswap -> MX_Only:MXOnly-1.25U-NoLED
- REF**: footprint MX_Only:MXOnly-2U-Hotswap -> MX_Only:MXOnly-2U-NoLED
- REF**: footprint MX_Only:MXOnly-7U-Hotswap-ReversedStabilizers -> MX_Only:MXOnly-7U-ReversedStabilizers-NoLED
- REF**: footprint MX_Only:MXOnly-2.25U-Hotswap -> MX_Only:MXOnly-2.25U-ReversedStabilizers-NoLED
- turned REF** to 0 degrees
- turned REF**13 to 0 degrees
- turned REF**14 to 0 degrees
Other:
- board size 405.1 x 105.1 mm -> 405.1 x 107.3 mm
- board text added: "Proto 6X"
